Commit message: deploy: update sim2real deployment models to latest DreamWaQ checkpoint (2026-09-02_20-58-03, iter 2999)

File: models/nxp_jaguar.urdf (robot description, URDF)
Before this commit: robot NXP_Jaguar, 15 links, 14 joints
Joints:
- joint Bl_hip_pitch_joint: limit lower=-3.14 upper=3.14 effort=14 velocity=20 -> lower=-3.14 upper=0.00 effort=14 velocity=20
- joint Br_hip_pitch_joint: limit lower=-3.14 upper=3.14 effort=14 velocity=20 -> lower=-3.14 upper=0.00 effort=14 velocity=20
- joint Fl_hip_pitch_joint: limit lower=-3.14 upper=3.14 effort=14 velocity=20 -> lower=-3.14 upper=0.00 effort=14 velocity=20
- joint Fr_hip_pitch_joint: limit lower=-3.14 upper=3.14 effort=14 velocity=20 -> lower=-3.14 upper=0.00 effort=14 velocity=20

Commit message: feat(models): update trained policy and checkpoint from nxp_jaguar_rough 2026-09-04_10-16-23 (iter 3499)
- Update production policy.pt and export policy.onnx from iter 3499
- Add checkpoint weights model_3499.pt, policy_3499.pt, and policy_3499.onnx
- Synchronize URDF joint limits for hip pitch [-1.80, 0.00] and knee [-0.10, 1.50]
- Update models/README.md documentation

File: models/nxp_jaguar.urdf (robot description, URDF)
Before this commit: robot NXP_Jaguar, 15 links, 14 joints
Joints:
- joint Bl_hip_pitch_joint: limit lower=-3.14 upper=0.00 effort=14 velocity=20 -> lower=-1.80 upper=0.00 effort=14 velocity=20
- joint Bl_knee_joint: limit lower=-0.10 upper=2.80 effort=14 velocity=20 -> lower=-0.10 upper=1.50 effort=14 velocity=20
- joint Br_hip_pitch_joint: limit lower=-3.14 upper=0.00 effort=14 velocity=20 -> lower=-1.80 upper=0.00 effort=14 velocity=20
- joint Br_knee_joint: limit lower=-0.10 upper=2.80 effort=14 velocity=20 -> lower=-0.10 upper=1.50 effort=14 velocity=20
- joint Fl_hip_pitch_joint: limit lower=-3.14 upper=0.00 effort=14 velocity=20 -> lower=-1.80 upper=0.00 effort=14 velocity=20
- joint Fl_knee_joint: limit lower=-0.10 upper=2.80 effort=14 velocity=20 -> lower=-0.10 upper=1.50 effort=14 velocity=20
- joint Fr_hip_pitch_joint: limit lower=-3.14 upper=0.00 effort=14 velocity=20 -> lower=-1.80 upper=0.00 effort=14 velocity=20
- joint Fr_knee_joint: limit lower=-0.10 upper=2.80 effort=14 velocity=20 -> lower=-0.10 upper=1.50 effort=14 velocity=20

File: urdf/nxp_jaguar.urdf (robot description, URDF)
Before this commit: robot NXP_Jaguar, 15 links, 14 joints
Joints:
- joint Bl_hip_pitch_joint: limit lower=-3.14 upper=3.14 effort=14 velocity=20 -> lower=-1.80 upper=0.00 effort=14 velocity=20
- joint Bl_knee_joint: limit lower=-0.10 upper=2.80 effort=14 velocity=20 -> lower=-0.10 upper=1.50 effort=14 velocity=20
- joint Br_hip_pitch_joint: limit lower=-3.14 upper=3.14 effort=14 velocity=20 -> lower=-1.80 upper=0.00 effort=14 velocity=20
- joint Br_knee_joint: limit lower=-0.10 upper=2.80 effort=14 velocity=20 -> lower=-0.10 upper=1.50 effort=14 velocity=20
- joint Fl_hip_pitch_joint: limit lower=-3.14 upper=3.14 effort=14 velocity=20 -> lower=-1.80 upper=0.00 effort=14 velocity=20
- joint Fl_knee_joint: limit lower=-0.10 upper=2.80 effort=14 velocity=20 -> lower=-0.10 upper=1.50 effort=14 velocity=20
- joint Fr_hip_pitch_joint: limit lower=-3.14 upper=3.14 effort=14 velocity=20 -> lower=-1.80 upper=0.00 effort=14 velocity=20
- joint Fr_knee_joint: limit lower=-0.10 upper=2.80 effort=14 velocity=20 -> lower=-0.10 upper=1.50 effort=14 velocity=20

Commit message: feat(sim2real): synchronize policy, foot contacts, standing pose, and actuator gains
- Deploy trained policy and weights from iteration 4999 (policy.pt, policy.onnx)
- Integrate Unitree-style spherical foot contacts (R=18.94mm, flush tangency) in URDF and MuJoCo
- Synchronize default standing joint angles with IsaacLab q0
- Align actuator gains (Kp=28.0 N*m/rad, Kd=0.7 N*m*s/rad) across CAN and controller configs
- Add urdf symlink to models/urdf for CMake and display launch compatibility
- Document foot contacts and tracking penalties in README

File: models/nxp_jaguar.urdf (robot description, URDF)
Before this commit: robot NXP_Jaguar, 15 links, 14 joints
Links:
- added link Bl_foot, mass 0.035; collision sphere radius=0.01894; visual sphere radius=0.01894
- added link Br_foot, mass 0.035; collision sphere radius=0.01894; visual sphere radius=0.01894
- added link Fl_foot, mass 0.035; collision sphere radius=0.01894; visual sphere radius=0.01894
- added link Fr_foot, mass 0.035; collision sphere radius=0.01894; visual sphere radius=0.01894
- link Bl_tibia_link: geometry collision box size=0.02 0.02 0.12; visual mesh filename=../meshes/Bl_tibia_pitch.STL
- link Br_tibia_link: geometry collision box size=0.02 0.02 0.12; visual mesh filename=../meshes/Br_tibia_pitch.STL
- link Fl_tibia_link: geometry collision box size=0.02 0.02 0.12; visual mesh filename=../meshes/Fl_tibia_pitch.STL
- link Fr_tibia_link: geometry collision box size=0.02 0.02 0.12; visual mesh filename=../meshes/Fr_tibia_pitch.STL
Joints:
- added joint Bl_foot_fixed: type fixed, parent Bl_tibia_link, child Bl_foot, origin xyz=0.1035 0.0175 -0.1445 rpy=0 0 0
- added joint Br_foot_fixed: type fixed, parent Br_tibia_link, child Br_foot, origin xyz=0.1035 -0.0175 -0.1445 rpy=0 0 0
- added joint Fl_foot_fixed: type fixed, parent Fl_tibia_link, child Fl_foot, origin xyz=0.1035 0.0175 -0.1445 rpy=0 0 0
- added joint Fr_foot_fixed: type fixed, parent Fr_tibia_link, child Fr_foot, origin xyz=0.1035 -0.0175 -0.1445 rpy=0 0 0
- joint Bl_hip_pitch_joint: origin xyz=-0.053 -0.005 0.000 rpy=0 0 0 -> xyz=-0.053 -0.005 0.000 rpy=0 0.20 0
- joint Bl_knee_joint: origin xyz=-0.157 0.0935 0.088 rpy=0 0 0 -> xyz=-0.157 0.0935 0.088 rpy=0 0.10 0
- joint Br_hip_pitch_joint: origin xyz=-0.053 -0.005 0.000 rpy=0 0 0 -> xyz=-0.053 -0.005 0.000 rpy=0 0.20 0
- joint Br_knee_joint: origin xyz=-0.157 -0.0935 0.088 rpy=0 0 0 -> xyz=-0.157 -0.0935 0.088 rpy=0 0.10 0
- joint Fl_hip_pitch_joint: origin xyz=0.053 -0.005 0.000 rpy=0 0 0 -> xyz=0.053 -0.005 0.000 rpy=0 0.20 0
- joint Fl_knee_joint: origin xyz=-0.157 0.0935 0.088 rpy=0 0 0 -> xyz=-0.157 0.0935 0.088 rpy=0 0.10 0
- joint Fr_hip_pitch_joint: origin xyz=0.053 -0.005 0.000 rpy=0 0 0 -> xyz=0.053 -0.005 0.000 rpy=0 0.20 0
- joint Fr_knee_joint: origin xyz=-0.157 -0.0935 0.088 rpy=0 0 0 -> xyz=-0.157 -0.0935 0.088 rpy=0 0.10 0

Commit message: feat(urdf): update distal foot pad collision geometry
Integrate authentic CAD distal foot pad extents and invisible collision
boxes in URDF and MuJoCo models.

File: models/nxp_jaguar.urdf (robot description, URDF)
Before this commit: robot NXP_Jaguar, 19 links, 18 joints
Links:
- link Bl_foot: geometry collision box size=0.046 0.035 0.018
- link Br_foot: geometry collision box size=0.046 0.035 0.018
- link Fl_foot: geometry collision box size=0.046 0.035 0.018
- link Fr_foot: geometry collision box size=0.046 0.035 0.018
Joints:
- joint Bl_foot_fixed: origin xyz=0.1035 0.0175 -0.1445 rpy=0 0 0 -> xyz=0.1035 0.0175 -0.1544 rpy=0 0 0
- joint Bl_hip_pitch_joint: limit lower=-1.80 upper=0.00 effort=14 velocity=20 -> lower=-3.14 upper=0.00 effort=14 velocity=20; origin xyz=-0.053 -0.005 0.000 rpy=0 0.20 0 -> xyz=-0.053 -0.005 0.000 rpy=0 0 0
- joint Bl_knee_joint: limit lower=-0.10 upper=1.50 effort=14 velocity=20 -> lower=-0.10 upper=2.80 effort=14 velocity=20; origin xyz=-0.157 0.0935 0.088 rpy=0 0.10 0 -> xyz=-0.157 0.0935 0.088 rpy=0 0 0
- joint Br_foot_fixed: origin xyz=0.1035 -0.0175 -0.1445 rpy=0 0 0 -> xyz=0.1035 -0.0175 -0.1544 rpy=0 0 0
- joint Br_hip_pitch_joint: limit lower=-1.80 upper=0.00 effort=14 velocity=20 -> lower=-3.14 upper=0.00 effort=14 velocity=20; origin xyz=-0.053 -0.005 0.000 rpy=0 0.20 0 -> xyz=-0.053 -0.005 0.000 rpy=0 0 0
- joint Br_knee_joint: limit lower=-0.10 upper=1.50 effort=14 velocity=20 -> lower=-0.10 upper=2.80 effort=14 velocity=20; origin xyz=-0.157 -0.0935 0.088 rpy=0 0.10 0 -> xyz=-0.157 -0.0935 0.088 rpy=0 0 0
- joint Fl_foot_fixed: origin xyz=0.1035 0.0175 -0.1445 rpy=0 0 0 -> xyz=0.1035 0.0175 -0.1544 rpy=0 0 0
- joint Fl_hip_pitch_joint: limit lower=-1.80 upper=0.00 effort=14 velocity=20 -> lower=-3.14 upper=0.00 effort=14 velocity=20; origin xyz=0.053 -0.005 0.000 rpy=0 0.20 0 -> xyz=0.053 -0.005 0.000 rpy=0 0 0
- joint Fl_knee_joint: limit lower=-0.10 upper=1.50 effort=14 velocity=20 -> lower=-0.10 upper=2.80 effort=14 velocity=20; origin xyz=-0.157 0.0935 0.088 rpy=0 0.10 0 -> xyz=-0.157 0.0935 0.088 rpy=0 0 0
- joint Fr_foot_fixed: origin xyz=0.1035 -0.0175 -0.1445 rpy=0 0 0 -> xyz=0.1035 -0.0175 -0.1544 rpy=0 0 0
- joint Fr_hip_pitch_joint: limit lower=-1.80 upper=0.00 effort=14 velocity=20 -> lower=-3.14 upper=0.00 effort=14 velocity=20; origin xyz=0.053 -0.005 0.000 rpy=0 0.20 0 -> xyz=0.053 -0.005 0.000 rpy=0 0 0
- joint Fr_knee_joint: limit lower=-0.10 upper=1.50 effort=14 velocity=20 -> lower=-0.10 upper=2.80 effort=14 velocity=20; origin xyz=-0.157 -0.0935 0.088 rpy=0 0.10 0 -> xyz=-0.157 -0.0935 0.088 rpy=0 0 0
